File: tce8.kicad_pcb (KiCad board)
At the start: 2 copper layers, 0 parts

Commit message: 1 bit alu
Parts:
- added NE555P_AUTO_CLOCK1: NE555P, Package_DIP:DIP-8_W7.62mm, F.Cu at (153.6, 91.2)
- added NE555P_MANUAL_CLOCK1: NE555P, Package_DIP:DIP-8_W7.62mm, F.Cu at (164.4, 91.2)
- added NE555P_SWITCH_MODE1: NE555P, Package_DIP:DIP-8_W7.62mm, F.Cu at (175.8, 91.2)
- added U1: 74LS32, Package_SO:SSOP-8_2.95x2.8mm_P0.65mm, F.Cu at (159.5, 57.7)
- added U1: 74LS32, Package_SO:SSOP-8_2.95x2.8mm_P0.65mm, F.Cu at (157.2, 70.4)
Routing:
- net (no net): track 0.00 -> 9.95 mm
- net Net-(U1-Pad5): track 0.00 -> 8.67 mm
- net Net-(U1-Pad4): track 0.00 -> 6.06 mm
- net SUB: track 0.00 -> 6.06 mm
- added copper zone on F.Cu, net (none)
- added copper zone on In2.Cu, net +5V
- added copper zone on In1.Cu, net GND
Other:
- board outline added: 243.8 x 304.8 mm
- copper layers 2 -> 4
