File: tce8.kicad_sch (KiCad schematic)
At the start: 0 parts

Commit message: 1 bit alu
Other:
- removed sheet ALU
- added sheet 1BitALU (one_bit_alu.kicad_sch)
- added sheet clock (clock.kicad_sch)
- added sheet program counter (program_counter.kicad_sch)
